File: Electronics/tactileSensor/tactileSensor.kicad_pcb (KiCad board)
At the start: 2 copper layers, 7 parts, among them J1 Conn_01x09_Pin

Commit message: PCB for mini sensor
Parts:
- removed C1, C2, C4: 100nF, Capacitor_SMD:C_Elec_3x5.4
- removed U2: ~, Package_LGA:ST_HLGA-10_2x2mm_P0.5mm_LayoutBorder3x2y
- C3: footprint Capacitor_SMD:C_Elec_3x5.4 -> Capacitor_SMD:C_0805_2012Metric; moved to B.Cu
- J1: value Conn_01x09_Pin -> Conn_01x07_Pin; footprint Connector_PinHeader_1.00mm:PinHeader_1x09_P1.00mm_Horizontal -> myOwn:padyBMP581
- moved U1 22.4 mm to (77.7, 121.3)
- moved C3 18.2 mm to (77.7, 121.0)
- moved J1 15.2 mm to (75.6, 119.8), turned to 0 degrees
Connections:
- J1 pad 2: 2 GND -> 5 SCK
- J1 pad 3: 3 CSB1 -> 2 GND
- J1 pad 4: 4 CSB2 -> 6 SDI
- J1 pad 5: 5 SCK -> 7 SDO
- J1 pad 6: 6 SDI -> 3 CSB1
- J1 pad 7: 7 SDO -> 2 GND
- U1 pad 7: 8 INT1 -> 2 GND
Routing:
- net 1 3V3: track 40.9 -> 6.73 mm, vias 0 -> 1
- net 2 GND: track 0.56 -> 9.32 mm, vias 0 -> 1
- net 3 CSB1: track 0.00 -> 2.68 mm
- net 5 SCK: track 0.00 -> 2.64 mm
- net 6 SDI: track 0.00 -> 1.95 mm
- net 7 SDO: track 2.52 -> 2.01 mm
Other:
- board outline added: 5 x 5 mm
